Commit message: Update Leo Rover dimensions from body drawing; account for LiDAR mounting pillars
URDF: body box 424x445x200mm, wheels 65mm wide at ±190mm track,
DiffDrive wheel_separation 0.380m, LiDAR at z=0.185m with enlarged
collision cylinder (r=60mm h=70mm) for pillar ring, min_range 0.18m.

Nav2: footprint [±0.212, ±0.223], padding 0.03, inflation_radius 0.45.
Explorer: obstacle_dist raised to 0.50m in all launch files and default.

Co-authored-by: langchengg <96649762+langchengg@users.noreply.github.com>

File: leo_exploration_ws/src/leo_exploration/urdf/leo_rover.urdf (robot description, URDF)
Before this commit: robot leo_rover, 7 links, 6 joints
Links:
- link base_link: geometry collision box size=0.424 0.445 0.200; visual box size=0.424 0.445 0.200
- link laser: geometry collision cylinder length=0.070 radius=0.060; visual cylinder length=0.040 radius=0.038
- link wheel_FL: geometry collision cylinder length=0.065 radius=0.065; visual cylinder length=0.065 radius=0.065
- link wheel_FR: geometry collision cylinder length=0.065 radius=0.065; visual cylinder length=0.065 radius=0.065
- link wheel_RL: geometry collision cylinder length=0.065 radius=0.065; visual cylinder length=0.065 radius=0.065
- link wheel_RR: geometry collision cylinder length=0.065 radius=0.065; visual cylinder length=0.065 radius=0.065
Joints:
- joint joint_FL: origin xyz=0.1475 0.213 0 rpy=0 0 0 -> xyz=0.1475 0.190 0 rpy=0 0 0
- joint joint_FR: origin xyz=0.1475 -0.213 0 rpy=0 0 0 -> xyz=0.1475 -0.190 0 rpy=0 0 0
- joint joint_RL: origin xyz=-0.1475 0.213 0 rpy=0 0 0 -> xyz=-0.1475 0.190 0 rpy=0 0 0
- joint joint_RR: origin xyz=-0.1475 -0.213 0 rpy=0 0 0 -> xyz=-0.1475 -0.190 0 rpy=0 0 0
- joint laser_joint: origin xyz=0.0 0.0 0.150 rpy=0 0 0 -> xyz=0.0 0.0 0.185 rpy=0 0 0

Commit message: v1

File: leo_exploration_ws/src/leo_exploration/urdf/leo_rover.urdf (robot description, URDF)
Before this commit: robot leo_rover, 7 links, 6 joints
Links:
- link base_link: geometry collision box size=0.445 0.289 0.092; visual box size=0.445 0.289 0.092
- link wheel_FL: geometry collision cylinder length=0.065 radius=0.0645; visual cylinder length=0.065 radius=0.0645
- link wheel_FR: geometry collision cylinder length=0.065 radius=0.0645; visual cylinder length=0.065 radius=0.0645
- link wheel_RL: geometry collision cylinder length=0.065 radius=0.0645; visual cylinder length=0.065 radius=0.0645
- link wheel_RR: geometry collision cylinder length=0.065 radius=0.0645; visual cylinder length=0.065 radius=0.0645
Joints:
- joint base_footprint_joint: origin xyz=0 0 0.065 rpy=0 0 0 -> xyz=0 0 0.0645 rpy=0 0 0
- joint joint_FL: origin xyz=0.1475 0.213 0 rpy=0 0 0 -> xyz=0.1475 0.1795 0 rpy=0 0 0
- joint joint_FR: origin xyz=0.1475 -0.213 0 rpy=0 0 0 -> xyz=0.1475 -0.1795 0 rpy=0 0 0
- joint joint_RL: origin xyz=-0.1475 0.213 0 rpy=0 0 0 -> xyz=-0.1475 0.1795 0 rpy=0 0 0
- joint joint_RR: origin xyz=-0.1475 -0.213 0 rpy=0 0 0 -> xyz=-0.1475 -0.1795 0 rpy=0 0 0
- joint laser_joint: origin xyz=0.0 0.0 0.150 rpy=0 0 0 -> xyz=0.0 0.0 0.1355 rpy=0 0 0

Commit message: imu

File: leo_exploration_ws/src/leo_exploration/urdf/leo_rover.urdf (robot description, URDF)
Before this commit: robot leo_rover, 7 links, 6 joints
Links:
- added link imu_link, mass 0.01
Joints:
- added joint imu_joint: type fixed, parent base_link, child imu_link, origin xyz=0 0 0.05 rpy=0 0 0
