Commit message: Fix typo in URDF
Co-authored-by: Copilot <copilot@github.com>

File: src/robot_description/urdf/mycobot_280pi/mycobot_280pi_arm.urdf.xacro (robot description, xacro)
@@ -41,5 +41,5 @@
         </geometry>
         <origin xyz="0.0 0 0" rpy="0 0 ${-pi}"/>
-      </visual>-
+      </visual>
       <collision>
         <geometry>
